File: pre-joulemeter-module.kicad_sch (KiCad schematic)
At the start: 0 parts

Commit message: Finished the schematic and added footprints
Parts:
- added C1: 100 uF, Capacitor_THT:C_Radial_D18.0mm_H35.5mm_P7.50mm, symbol Device:C
- added D1: 1N5400, Diode_THT:D_DO-201AD_P15.24mm_Horizontal, symbol Diode:1N5400
- added D2: LED_Small, LED_SMD:LED_1812_4532Metric_Pad1.30x3.40mm_HandSolder, symbol Device:LED_Small
- added J1, J2, J3: Conn_01x02, Connector_AMASS:AMASS_XT60PW-M_1x02_P7.20mm_Horizontal, symbol Connector_Generic:Conn_01x02
- added R1: R, Resistor_SMD:R_1812_4532Metric_Pad1.30x3.40mm_HandSolder, symbol Device:R
Connections:
- new net: D2.2 (A), R1.1
- new net +BATT: C1.1, D1.1 (K), J1.2 (Pin_2), J2.2 (Pin_2), J3.2 (Pin_2), R1.2
- new net GNDPWR: C1.2, D1.2 (A), D2.1 (K), J1.1 (Pin_1), J2.1 (Pin_1), J3.1 (Pin_1)
